Commit message: add: joint pos,vel plots

File: workspace/models/SO101/so101_new_calib.urdf (robot description, URDF)
Before this commit: robot so101_new_calib, 8 links, 7 joints
Joints:
- joint elbow_flex: limit lower=-1.69 upper=1.69 effort=10 velocity=10 -> lower=-1.69 upper=1.69 effort=10 velocity=3.14
- joint gripper: limit lower=-0.174533 upper=1.74533 effort=10 velocity=10 -> lower=-0.174533 upper=1.74533 effort=10 velocity=3.14
- joint shoulder_lift: limit lower=-1.74533 upper=1.74533 effort=10 velocity=10 -> lower=-1.74533 upper=1.74533 effort=10 velocity=3.14
- joint shoulder_pan: limit lower=-1.91986 upper=1.91986 effort=10 velocity=10 -> lower=-1.91986 upper=1.91986 effort=10 velocity=3.14
- joint wrist_flex: limit lower=-1.65806 upper=1.65806 effort=10 velocity=10 -> lower=-1.65806 upper=1.65806 effort=10 velocity=3.14
- joint wrist_roll: limit lower=-2.74385 upper=2.84121 effort=10 velocity=10 -> lower=-2.74385 upper=2.84121 effort=10 velocity=3.14
